Commit message: Working initial integration with MMP

File: src/kortex_description/arms/gen3/urdf/gen3_macro.xacro (robot description, xacro)
@@ -48,18 +48,4 @@
       </collision>
     </link>
-    <joint
-      name="joint_1"
-      type="continuous">
-      <origin xyz="0 0 0.15643" rpy="3.1416 2.7629E-18 -4.9305E-36" />
-      <parent
-        link="base_link" />
-      <child
-        link="shoulder_link" />
-      <axis
-        xyz="0 0 1" />
-      <limit
-        effort="39"
-        velocity="0.8727" />
-    </joint>
     <link name="half_arm_1_link">
       <inertial>
@@ -84,4 +70,129 @@
       </collision>
     </link>
+    <link name="half_arm_2_link">
+      <inertial>
+        <origin xyz="-4.4E-05 -0.006641 -0.117892" rpy="0 0 0" />
+        <mass value="1.1636" />
+        <inertia ixx="0.010932" ixy="0" ixz="-7E-06" iyy="0.011127" iyz="0.000606" izz="0.001043" />
+      </inertial>
+      <visual>
+        <origin xyz="0 0 0" rpy="0 0 0" />
+        <geometry>
+          <mesh filename="package://kortex_description/arms/gen3/meshes/half_arm_2_link.STL" />
+        </geometry>
+        <material name="">
+          <color rgba="0.75294 0.75294 0.75294 1" />
+        </material>
+      </visual>
+      <collision>
+        <origin xyz="0 0 0" rpy="0 0 0" />
+        <geometry>
+          <mesh filename="package://kortex_description/arms/gen3/meshes/half_arm_2_link.STL" />
+        </geometry>
+      </collision>
+    </link>
+    <link name="forearm_link">
+      <inertial>
+        <origin xyz="-1.8E-05 -0.075478 -0.015006" rpy="0 0 0" />
+        <mass value="0.9302" />
+        <inertia ixx="0.008147" ixy="-1E-06" ixz="0" iyy="0.000631" iyz="-0.0005" izz="0.008316" />
+      </inertial>
+      <visual>
+        <origin xyz="0 0 0" rpy="0 0 0" />
+        <geometry>
+          <mesh filename="package://kortex_description/arms/gen3/meshes/forearm_link.STL" />
+        </geometry>
+        <material name="">
+          <color rgba="0.75294 0.75294 0.75294 1" />
+        </material>
+      </visual>
+      <collision>
+        <origin xyz="0 0 0" rpy="0 0 0" />
+        <geometry>
+          <mesh filename="package://kortex_description/arms/gen3/meshes/forearm_link.STL" />
+        </geometry>
+      </collision>
+    </link>
+    <link name="spherical_wrist_1_link">
+      <inertial>
+        <origin xyz="1E-06 -0.009432 -0.063883" rpy="0 0 0" />
+        <mass value="0.6781" />
+        <inertia ixx="0.001596" ixy="0" ixz="0" iyy="0.001607" iyz="0.000256" izz="0.000399" />
+      </inertial>
+      <visual>
+        <origin xyz="0 0 0" rpy="0 0 0" />
+        <geometry>
+          <mesh filename="package://kortex_description/arms/gen3/meshes/spherical_wrist_1_link.STL" />
+        </geometry>
+        <material name="">
+          <color rgba="0.75294 0.75294 0.75294 1" />
+        </material>
+      </visual>
+      <collision>
+        <origin xyz="0 0 0" rpy="0 0 0" />
+        <geometry>
+          <mesh filename="package://kortex_description/arms/gen3/meshes/spherical_wrist_1_link.STL" />
+        </geometry>
+      </collision>
+    </link>
+    <link name="spherical_wrist_2_link">
+      <inertial>
+        <origin xyz="1E-06 -0.045483 -0.00965" rpy="0 0 0" />
+        <mass value="0.6781" />
+        <inertia ixx="0.001641" ixy="0" ixz="0" iyy="0.00041" iyz="-0.000278" izz="0.001641" />
+      </inertial>
+      <visual>
+        <origin xyz="0 0 0" rpy="0 0 0" />
+        <geometry>
+          <mesh filename="package://kortex_description/arms/gen3/meshes/spherical_wrist_2_link.STL" />
+        </geometry>
+        <material name="">
+          <color rgba="0.75294 0.75294 0.75294 1" />
+        </material>
+      </visual>
+      <collision>
+        <origin xyz="0 0 0" rpy="0 0 0" />
+        <geometry>
+          <mesh filename="package://kortex_description/arms/gen3/meshes/spherical_wrist_2_link.STL" />
+        </geometry>
+      </collision>
+    </link>
+    <link name="bracelet_link">
+      <inertial>
+        <origin xyz="-0.000281 -0.011402 -0.029798" rpy="0 0 0" />
+        <mass value="0.5006" />
+        <inertia ixx="0.000587" ixy="3E-06" ixz="3E-06" iyy="0.000369" iyz="0.000118" izz="0.000609" />
+      </inertial>
+      <visual>
+        <origin xyz="0 0 0" rpy="0 0 0" />
+        <geometry>
+          <mesh filename="package://kortex_description/arms/gen3/meshes/bracelet_link.STL" />
+        </geometry>
+        <material name="">
+          <color rgba="0.75294 0.75294 0.75294 1" />
+        </material>
+      </visual>
+      <collision>
+        <origin xyz="0 0 0" rpy="0 0 0" />
+        <geometry>
+          <mesh filename="package://kortex_description/arms/gen3/meshes/bracelet_link.STL" />
+        </geometry>
+      </collision>
+    </link>
+    <link name="end_effector_link" />
+    <joint
+      name="joint_1"
+      type="continuous">
+      <origin xyz="0 0 0.15643" rpy="3.1416 2.7629E-18 -4.9305E-36" />
+      <parent
+        link="base_link" />
+      <child
+        link="shoulder_link" />
+      <axis
+        xyz="0 0 1" />
+      <limit
+        effort="39"
+        velocity="0.8727" />
+    </joint>
     <joint
       name="joint_2"
@@ -97,26 +208,4 @@
       <limit lower="-2.1" upper="2.1" effort="39" velocity="0.8727" />
     </joint>
-    <link name="half_arm_2_link">
-      <inertial>
-        <origin xyz="-4.4E-05 -0.006641 -0.117892" rpy="0 0 0" />
-        <mass value="1.1636" />
-        <inertia ixx="0.010932" ixy="0" ixz="-7E-06" iyy="0.011127" iyz="0.000606" izz="0.001043" />
-      </inertial>
-      <visual>
-        <origin xyz="0 0 0" rpy="0 0 0" />
-        <geometry>
-          <mesh filename="package://kortex_description/arms/gen3/meshes/half_arm_2_link.STL" />
-        </geometry>
-        <material name="">
-          <color rgba="0.75294 0.75294 0.75294 1" />
-        </material>
-      </visual>
-      <collision>
-        <origin xyz="0 0 0" rpy="0 0 0" />
-        <geometry>
-          <mesh filename="package://kortex_description/arms/gen3/meshes/half_arm_2_link.STL" />
-        </geometry>
-      </collision>
-    </link>
     <joint
       name="joint_3"
@@ -133,26 +222,4 @@
         velocity="0.8727" />
     </joint>
-    <link name="forearm_link">
-      <inertial>
-        <origin xyz="-1.8E-05 -0.075478 -0.015006" rpy="0 0 0" />
-        <mass value="0.9302" />
-        <inertia ixx="0.008147" ixy="-1E-06" ixz="0" iyy="0.000631" iyz="-0.0005" izz="0.008316" />
-      </inertial>
-      <visual>
-        <origin xyz="0 0 0" rpy="0 0 0" />
-        <geometry>
-          <mesh filename="package://kortex_description/arms/gen3/meshes/forearm_link.STL" />
-        </geometry>
-        <material name="">
-          <color rgba="0.75294 0.75294 0.75294 1" />
-        </material>
-      </visual>
-      <collision>
-        <origin xyz="0 0 0" rpy="0 0 0" />
-        <geometry>
-          <mesh filename="package://kortex_description/arms/gen3/meshes/forearm_link.STL" />
-        </geometry>
-      </collision>
-    </link>
     <joint
       name="joint_4"
@@ -168,26 +235,4 @@
       <limit lower="-2.4" upper="2.4" effort="39" velocity="0.8727" />
     </joint>
-    <link name="spherical_wrist_1_link">
-      <inertial>
-        <origin xyz="1E-06 -0.009432 -0.063883" rpy="0 0 0" />
-        <mass value="0.6781" />
-        <inertia ixx="0.001596" ixy="0" ixz="0" iyy="0.001607" iyz="0.000256" izz="0.000399" />
-      </inertial>
-      <visual>
-        <origin xyz="0 0 0" rpy="0 0 0" />
-        <geometry>
-          <mesh filename="package://kortex_description/arms/gen3/meshes/spherical_wrist_1_link.STL" />
-        </geometry>
-        <material name="">
-          <color rgba="0.75294 0.75294 0.75294 1" />
-        </material>
-      </visual>
-      <collision>
-        <origin xyz="0 0 0" rpy="0 0 0" />
-        <geometry>
-          <mesh filename="package://kortex_description/arms/gen3/meshes/spherical_wrist_1_link.STL" />
-        </geometry>
-      </collision>
-    </link>
     <joint
       name="joint_5"
@@ -204,26 +249,4 @@
         velocity="0.8727" />
     </joint>
-    <link name="spherical_wrist_2_link">
-      <inertial>
-        <origin xyz="1E-06 -0.045483 -0.00965" rpy="0 0 0" />
-        <mass value="0.6781" />
-        <inertia ixx="0.001641" ixy="0" ixz="0" iyy="0.00041" iyz="-0.000278" izz="0.001641" />
-      </inertial>
-      <visual>
-        <origin xyz="0 0 0" rpy="0 0 0" />
-        <geometry>
-          <mesh filename="package://kortex_description/arms/gen3/meshes/spherical_wrist_2_link.STL" />
-        </geometry>
-        <material name="">
-          <color rgba="0.75294 0.75294 0.75294 1" />
-        </material>
-      </visual>
-      <collision>
-        <origin xyz="0 0 0" rpy="0 0 0" />
-        <geometry>
-          <mesh filename="package://kortex_description/arms/gen3/meshes/spherical_wrist_2_link.STL" />
-        </geometry>
-      </collision>
-    </link>
     <joint
       name="joint_6"
@@ -239,26 +262,4 @@
       <limit lower="-1.9" upper="1.9" effort="9" velocity="0.8727" />
     </joint>
-    <link name="bracelet_link">
-      <inertial>
-        <origin xyz="-0.000281 -0.011402 -0.029798" rpy="0 0 0" />
-        <mass value="0.5006" />
-        <inertia ixx="0.000587" ixy="3E-06" ixz="3E-06" iyy="0.000369" iyz="0.000118" izz="0.000609" />
-      </inertial>
-      <visual>
-        <origin xyz="0 0 0" rpy="0 0 0" />
-        <geometry>
-          <mesh filename="package://kortex_description/arms/gen3/meshes/bracelet_link.STL" />
-        </geometry>
-        <material name="">
-          <color rgba="0.75294 0.75294 0.75294 1" />
-        </material>
-      </visual>
-      <collision>
-        <origin xyz="0 0 0" rpy="0 0 0" />
-        <geometry>
-          <mesh filename="package://kortex_description/arms/gen3/meshes/bracelet_link.STL" />
-        </geometry>
-      </collision>
-    </link>
     <joint
       name="joint_7"
@@ -275,5 +276,4 @@
         velocity="0.8727" />
     </joint>
-    <link name="end_effector_link" />
     <joint
       name="end_effector"

Commit message: Better integration with sai2, added ori control

File: src/kortex_description/arms/gen3/urdf/gen3_macro.xacro (robot description, xacro)
@@ -181,7 +181,5 @@
     </link>
     <link name="end_effector_link" />
-    <joint
-      name="joint_1"
-      type="continuous">
+    <joint name="joint_1" type="continuous">
       <origin xyz="0 0 0.15643" rpy="3.1416 2.7629E-18 -4.9305E-36" />
       <parent
@@ -195,7 +193,5 @@
         velocity="0.8727" />
     </joint>
-    <joint
-      name="joint_2"
-      type="revolute">
+    <joint name="joint_2" type="revolute">
       <origin xyz="0 0.005375 -0.12838" rpy="1.5708 2.1343E-17 -1.1102E-16" />
       <parent
@@ -208,7 +204,5 @@
       <limit lower="-2.1" upper="2.1" effort="39" velocity="0.8727" />
     </joint>
-    <joint
-      name="joint_3"
-      type="continuous">
+    <joint name="joint_3" type="continuous">
       <origin xyz="0 -0.21038 -0.006375" rpy="-1.5708 1.2326E-32 -2.9122E-16" />
       <parent
@@ -222,7 +216,5 @@
         velocity="0.8727" />
     </joint>
-    <joint
-      name="joint_4"
-      type="revolute">
+    <joint name="joint_4" type="revolute">
       <origin xyz="0 0.006375 -0.21038" rpy="1.5708 -6.6954E-17 -1.6653E-16" />
       <parent
@@ -235,7 +227,5 @@
       <limit lower="-2.4" upper="2.4" effort="39" velocity="0.8727" />
     </joint>
-    <joint
-      name="joint_5"
-      type="continuous">
+    <joint name="joint_5" type="continuous">
       <origin xyz="0 -0.20843 -0.006375" rpy="-1.5708 2.2204E-16 -6.373E-17" />
       <parent
@@ -249,7 +239,5 @@
         velocity="0.8727" />
     </joint>
-    <joint
-      name="joint_6"
-      type="revolute">
+    <joint name="joint_6" type="revolute">
       <origin xyz="0 0.00017505 -0.10593" rpy="1.5708 9.2076E-28 -8.2157E-15" />
       <parent
@@ -262,7 +250,5 @@
       <limit lower="-1.9" upper="1.9" effort="9" velocity="0.8727" />
     </joint>
-    <joint
-      name="joint_7"
-      type="continuous">
+    <joint name="joint_7" type="continuous">
       <origin xyz="0 -0.10593 -0.00017505" rpy="-1.5708 -5.5511E-17 9.6396E-17" />
       <parent
@@ -276,8 +262,6 @@
         velocity="0.8727" />
     </joint>
-    <joint
-      name="end_effector"
-      type="fixed">
-      <origin xyz="0 0 -0.0615250000000001" rpy="3.14159265358979 1.09937075168372E-32 0" />
+    <joint name="end_effector" type="fixed">
+      <origin xyz="0 0 -0.0615250000000001" rpy="0 0 0" />
       <parent
         link="bracelet_link" />

File: src/kortex_description/arms/mmp/urdf/mmp_macro.xacro (robot description, xacro)
@@ -4,4 +4,5 @@
   <xacro:property name="last_arm_link" value="end_effector_link"/>
   <xacro:macro name="load_arm" params="parent:='' *origin">
+     <!-- GROUND LINK -->
      <link name="base_link">
         <visual>
@@ -21,4 +22,5 @@
         </collision> -->
     </link>
+    <!-- MOBILE BASE LINKS -->
     <link name="x_prismatic">
         <visual>
@@ -55,14 +57,15 @@
         </collision> -->
     </link>
+      <!-- MOBILE BASE + LINK 0 OF KINOVA ARM -->
       <link name="mmp_base">
         <inertial>
-          <origin xyz="-0.000648 -0.000166 0.084487" rpy="0 0 0" />
-          <mass value="1.697" />
-          <inertia ixx="0.004622" ixy="9E-06" ixz="6E-05" iyy="0.004495" iyz="9E-06" izz="0.002079" />
+          <origin xyz="0.0 0.0 0.1757" rpy="0 0 0" />
+          <mass value="64.6" />
+          <inertia ixx="1.721" ixy="0.0" ixz="0.0" iyy="1.712" iyz="0.0" izz="2.030" />
         </inertial>
         <visual>
           <origin xyz="0 0 0" rpy="0 0 0" />
           <geometry>
-            <mesh filename="package://kortex_description/arms/gen3/meshes/base_link.STL" />
+            <mesh filename="package://kortex_description/arms/mmp/meshes/BaseCombo.STL" />
           </geometry>
           <material name="">
@@ -73,5 +76,5 @@
           <origin xyz="0 0 0" rpy="0 0 0" />
           <geometry>
-            <mesh filename="package://kortex_description/arms/gen3/meshes/base_link.STL" />
+            <mesh filename="package://kortex_description/arms/mmp/meshes/BaseCombo.STL" />
           </geometry>
         </collision>
@@ -232,7 +235,5 @@
     </link>
     <link name="end_effector_link" />
-    <joint
-      name="joint_1"
-      type="prismatic">
+    <joint name="joint_1" type="prismatic">
       <origin xyz="0 0 0" rpy="0 0 0" />
       <parent
@@ -244,7 +245,5 @@
       <limit lower="-2.1" upper="2.1" effort="39" velocity="0.8727" />
     </joint>
-    <joint
-      name="joint_2"
-      type="prismatic">
+    <joint name="joint_2" type="prismatic">
       <origin xyz="0 0 0" rpy="0 0 0" />
       <parent
@@ -256,7 +255,5 @@
       <limit lower="-2.1" upper="2.1" effort="39" velocity="0.8727" />
     </joint>
-    <joint
-      name="joint_3"
-      type="continuous">
+    <joint name="joint_3" type="continuous">
       <origin xyz="0 0 0" rpy="0 0 0" />
       <parent
@@ -270,8 +267,6 @@
         velocity="0.8727" />
     </joint>
-    <joint
-      name="joint_4"
-      type="continuous">
-      <origin xyz="0 0 0.15643" rpy="3.1416 2.7629E-18 -4.9305E-36" />
+    <joint name="joint_4" type="continuous">
+      <origin xyz="0 0 0.48643" rpy="3.1416 2.7629E-18 -3.14" />
       <parent
         link="mmp_base" />
@@ -284,7 +279,5 @@
         velocity="0.8727" />
     </joint>
-    <joint
-      name="joint_5"
-      type="revolute">
+    <joint name="joint_5" type="revolute">
       <origin xyz="0 0.005375 -0.12838" rpy="1.5708 2.1343E-17 -1.1102E-16" />
       <parent
@@ -297,7 +290,5 @@
       <limit lower="-2.1" upper="2.1" effort="39" velocity="0.8727" />
     </joint>
-    <joint
-      name="joint_6"
-      type="continuous">
+    <joint name="joint_6" type="continuous">
       <origin xyz="0 -0.21038 -0.006375" rpy="-1.5708 1.2326E-32 -2.9122E-16" />
       <parent
@@ -311,7 +302,5 @@
         velocity="0.8727" />
     </joint>
-    <joint
-      name="joint_7"
-      type="revolute">
+    <joint name="joint_7" type="revolute">
       <origin xyz="0 0.006375 -0.21038" rpy="1.5708 -6.6954E-17 -1.6653E-16" />
       <parent
@@ -322,9 +311,7 @@
         xyz="0 0 1" />
       <!-- <limit lower="-2.66" upper="2.66" effort="39" velocity="0.8727" /> -->
-      <limit lower="-2.4" upper="2.4" effort="39" velocity="0.8727" />
-    </joint>
-    <joint
-      name="joint_8"
-      type="continuous">
+      <limit lower="-2.1" upper="2.1" effort="39" velocity="0.8727" />
+    </joint>
+    <joint name="joint_8" type="continuous">
       <origin xyz="0 -0.20843 -0.006375" rpy="-1.5708 2.2204E-16 -6.373E-17" />
       <parent
@@ -338,7 +325,5 @@
         velocity="0.8727" />
     </joint>
-    <joint
-      name="joint_9"
-      type="revolute">
+    <joint name="joint_9" type="revolute">
       <origin xyz="0 0.00017505 -0.10593" rpy="1.5708 9.2076E-28 -8.2157E-15" />
       <parent
@@ -351,7 +336,5 @@
       <limit lower="-1.9" upper="1.9" effort="9" velocity="0.8727" />
     </joint>
-    <joint
-      name="joint_10"
-      type="continuous">
+    <joint name="joint_10" type="continuous">
       <origin xyz="0 -0.10593 -0.00017505" rpy="-1.5708 -5.5511E-17 9.6396E-17" />
       <parent
@@ -365,8 +348,6 @@
         velocity="0.8727" />
     </joint>
-    <joint
-      name="end_effector"
-      type="fixed">
-      <origin xyz="0 0 -0.0615250000000001" rpy="3.14159265358979 1.09937075168372E-32 0" />
+    <joint name="end_effector" type="fixed">
+      <origin xyz="0 0 -0.0615250000000001" rpy="0 0 0" />
       <parent
         link="bracelet_link" />
